File: schematics/base-station/peeler_mouse_schematic.kicad_sch (KiCad schematic)
At the start: 11 parts, among them M1 Larger Unident Bipolar Stepper, M2 Smallr Unident Bipolar Stepper, SW1 Yellow, SW2 Green, SW3 Blue, SW4 Black

Commit message: chore: update base station schematic
Parts:
- removed A1: Arduino_Nano_v3.x, Module:Arduino_Nano, symbol MCU_Module:Arduino_Nano_v3.x
- added MT1: PEC11R-4215F-S0024, PEC11R-4215F-S0024:XDCR_PEC11R-4215F-S0024, symbol encoder:PEC11R-4215F-S0024
- added U1: OLED2.42" SSD1309, OLED_SSD1309:OLED_SSD1309, symbol ssd1309:OLED_SSD1309_1
- added U2: NUCLEO-H753ZI, NUCLEO-H753ZI:MODULE_NUCLEO-H753ZI, symbol stm32:NUCLEO-H753ZI
- added X1: (no value), symbol stm32:POWER
- added X2: (no value), symbol library:UART
- SD1, SD2: value ~ -> (none)
Connections:
- net at PS1.3 (-Vo), PS2.1 (-Vin), PS2.3 (-Vout)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: now also MT1.1, MT1.COM, U1.1 (GND), X1. (GND)
- net Button A: now reaches SW1.2
- net Button A: now also U2.CN9_4 (D52/USART_B_RX)
- net Button B: now reaches SW2.2
- net Button B: now also U2.CN9_6 (D53/USART_B_TX)
- net Button C: now reaches SW3.2
- net Button C: now also U2.CN9_8 (D54/USART_B_RTS)
- net LIN STEP: now reaches SD1. (PUL-)
- net LIN STEP: now also U2.CN7_1 (D16/I2S_A_MCK)
- net Button D: now reaches SW4.2
- net Button D: now also U2.CN9_2 (D51/USART_B_SCLK)
- net at PS2.4 (+Vout): now also U1.2 (VCC), X1. (GND)
- net ROT STEP: now reaches SD2. (PUL-)
- net ROT STEP: now also U2.CN10_14 (D1/USART_A_TX)
- new net: MT1.S1 (SHIELD), MT1.S2 (SHIELD)
- new net Button Enc: MT1.2, U2.CN9_10 (D55/USART_B_CTS)
- new net GND_CN10: U2.CN10_17 (GND_CN10), U2.CN10_22 (GND_CN10), U2.CN10_27 (GND_CN10), U2.CN10_5 (GND_CN10)
- new net GND_CN8: U2.CN8_11 (GND_CN8), U2.CN8_13 (GND_CN8)
- new net GND_CN9: U2.CN9_12 (GND_CN9), U2.CN9_23 (GND_CN9)
- new net LCD SCL: U1.3 (SCK), U2.CN9_19 (D69/I2C_B_SCL)
- new net LCD SDA: U1.4 (SDA), U2.CN9_21 (D68/I2C_B_SDA)
- new net LIN DIR: SD1. (PUL-), U2.CN9_24 (D61/SAI_B_SCK)
- new net ROT DIR: SD2. (PUL-), U2.CN9_28 (D63/SAI_B_FS)
- new net encoder ch1: MT1.A, U2.CN7_12 (D12/SPI_A_MISO)
- new net encoder ch2: MT1.B, U2.CN7_13 (D22/I2S_B_SD/SPI_B_MOSI)
- new net rx: U2.CN10_34 (D35/TIMER_C_PWM3), X2. (RX)
- new net tx: U2.CN10_32 (D36/TIMER_C_PWM2), X2. (RX)
Other:
- note added: "ETHERNET"
- note added: "NUCLEO-H753ZI"
- note added: "Note: Follow Pin Names (ie. D11), not pin locations!"
- note added: "USB OTG"
- note added: "USB ST-LINK"
- company: (none) -> Saxion SMART
- title: (none) -> Cable Peeler Base Station
- moved on the sheet: PS1, PS2
