File: schematics/cutting-head/.history/kabelPeeler v1.1.kicad_sch (KiCad schematic)
At the start: 60 parts, among them J1 Steppermotor, J2 Main input, J3 Limit switch, J4 Encoder, J5 LED-Output, J6 Ext Motor VCC, Q1 FDV301N, U1 XIAO-ESP32-S3-DIP, U2 TMC2209, U5 AMS1117-5.0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

Commit message: feat: cutting-head schematic v1.1
Parts:
- removed U8: R-78B3.3-2.0, Converter_DCDC:Converter_DCDC_RECOM_R-78B-2.0_THT, symbol Converter_DCDC:R-78B3.3-2.0
- removed U9: R-78B5.0-2.0, Converter_DCDC:Converter_DCDC_RECOM_R-78B-2.0_THT, symbol Converter_DCDC:R-78B5.0-2.0
- added Q2: AO3401A, Package_TO_SOT_SMD:SOT-23, symbol Transistor_FET:AO3401A
- added R3: 10K, Resistor_SMD:R_0805_2012Metric_Pad1.20x1.40mm_HandSolder, symbol Device:R
- C8: value 100nF -> 10nF
- R4: value 2.2K -> 1.5K
- R5: value 2.2K -> 1K
- R8: value 0 -> NC
- TP1, TP10, TP11, TP2, TP3, TP4, TP5, TP6, TP7, TP8, TP9: footprint TestPoint:TestPoint_Pad_D1.5mm -> TestPoint:TestPoint_Pad_D1.0mm
Connections:
- net +3.3V: now also Q2.2 (S)
- net +3V3: now also Q2.3 (D)
- net GND: now also R3.1
- net VBUS: now also Q2.1 (G), R3.2
Other:
- note removed: "Optional: through-hole dc/dc replacements"
- moved on the sheet: D1, D2, Q1, R2, R4, R5, R6, TP1, TP10, TP11, TP2
